File: BMSv2/BMSv2.kicad_sch (KiCad schematic)
At the start: 122 parts, among them J2 Conn_01x04_Socket, J3 Conn_01x02_Pin, J4 Conn_01x02_Pin, J5 Conn_01x03_Pin, Q1 AO3401A, SW1 SW_BOOT0, U1 STM32F405RGTx, U2 MCP2561-E-SN, U4 MP2332H, U5 AMS1117-3.3

Commit message: Add files via upload
Connections:
- net +3V3 is gone; now on net +3.3V: J2.3 (Pin_3), R1.1, R2.1, R3.1, R4.1
Changed lines of the file:
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@@
     )
   )
-  (symbol (lib_id "power:+3V3") (at 272.669 30.099 0) (unit 1)
-    (in_bom yes) (on_board yes) (dnp no) (fields_autoplaced)
-    (property "Reference" "#PWR01" (at 272.669 33.909 0)
-      (effects (font (size 1.27 1.27)) hide)
-    )
-    (property "Value" "+3V3" (at 272.669 25.019 0)
-      (effects (font (size 1.27 1.27)))
-    )
-    (property "Footprint" "" (at 272.669 30.099 0)
-      (effects (font (size 1.27 1.27)) hide)
-    )
-    (property "Datasheet" "" (at 272.669 30.099 0)
-      (effects (font (size 1.27 1.27)) hide)
-    )
-    (pin "1")
-    (instances
-      (project "BMSv2"
-        (path "/a5c08c1c-7045-4a3a-8914-115fdd89801e"
-          (reference "#PWR01") (unit 1)
-        )
-      )
-    )
-  )
   (symbol (lib_id "Device:C") (at 38.9135 121.1065 0) (unit 1)
     (in_bom yes) (on_board yes) (dnp no)
@@
     )
   )
+  (symbol (lib_id "power:+3.3V") (at 272.669 30.099 0) (unit 1)
+    (in_bom yes) (on_board yes) (dnp no) (fields_autoplaced)
+    (property "Reference" "#PWR01" (at 272.669 33.909 0)
+      (effects (font (size 1.27 1.27)) hide)
+    )
+    (property "Value" "+3.3V" (at 272.669 25.527 0)
+      (effects (font (size 1.27 1.27)))
+    )
+    (property "Footprint" "" (at 272.669 30.099 0)
+      (effects (font (size 1.27 1.27)) hide)
+    )
+    (property "Datasheet" "" (at 272.669 30.099 0)
+      (effects (font (size 1.27 1.27)) hide)
+    )
+    (pin "1")
+    (instances
+      (project "BMSv2"
+        (path "/a5c08c1c-7045-4a3a-8914-115fdd89801e"
+          (reference "#PWR01") (unit 1)
+        )
+      )
+    )
+  )
   (symbol (lib_id "power:+3.3V") (at 376.936 163.195 0) (unit 1)
     (in_bom yes) (on_board yes) (dnp no)
@@
     )
   )
+  (symbol (lib_id "power:+3.3V") (at 141.224 86.106 90) (unit 1)
+    (in_bom yes) (on_board yes) (dnp no) (fields_autoplaced)
+    (property "Reference" "#PWR049" (at 145.034 86.106 0)
+      (effects (font (size 1.27 1.27)) hide)
+    )
+    (property "Value" "+3.3V" (at 137.795 86.106 90)
+      (effects (font (size 1.27 1.27)) (justify left))
+    )
+    (property "Footprint" "" (at 141.224 86.106 0)
+      (effects (font (size 1.27 1.27)) hide)
+    )
+    (property "Datasheet" "" (at 141.224 86.106 0)
+      (effects (font (size 1.27 1.27)) hide)
+    )
+    (pin "1")
+    (instances
+      (project "BMSv2"
+        (path "/a5c08c1c-7045-4a3a-8914-115fdd89801e"
+          (reference "#PWR049") (unit 1)
+        )
+      )
+    )
+  )
   (symbol (lib_id "Device:LED") (at 267.589 114.681 270) (mirror x) (unit 1)
     (in_bom yes) (on_board yes) (dnp no) (fields_autoplaced)
@@
         )
       )
-    )
-  )
-  (symbol (lib_id "power:+3V3") (at 141.224 86.106 90) (unit 1)
-    (in_bom yes) (on_board yes) (dnp no) (fields_autoplaced)
-    (property "Reference" "#PWR049" (at 145.034 86.106 0)
-      (effects (font (size 1.27 1.27)) hide)
-    )
-    (property "Value" "+3V3" (at 137.1346 86.106 90)
-      (effects (font (size 1.27 1.27)) (justify left))
-    )
-    (property "Footprint" "" (at 141.224 86.106 0)
-      (effects (font (size 1.27 1.27)) hide)
-    )
-    (property "Datasheet" "" (at 141.224 86.106 0)
-      (effects (font (size 1.27 1.27)) hide)
-    )
-    (pin "1")
-    (instances
-      (project "BMSv2"
-        (path "/a5c08c1c-7045-4a3a-8914-115fdd89801e"
-          (reference "#PWR049") (unit 1)
-        )
-      )
