File: BMSv2/Malo_scieżęk.kicad_pcb (KiCad board)
At the start: 2 copper layers, 122 parts, among them J1 Conn_01x05, J2 Conn_01x04_Socket, J3 Conn_01x02_Pin, J4 Conn_01x02_Pin, J5 Conn_01x03_Pin, Q1 AO3401A, Q10 MMBT3904, Q11 MMBT3904, Q12 MMBT3904, Q13 MMBT3904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

Commit message: Add files via upload
Parts:
- moved J1 68.8 mm to (188.4, 79.3)
- moved C25 67.8 mm to (181.3, 61.3)
- moved C26 67.8 mm to (181.6, 69.5)
- moved C27 67.8 mm to (181.5, 76.5)
- moved D3 67.8 mm to (167.5, 65.9)
- moved D4 67.8 mm to (167.5, 74.2)
- moved D5 67.8 mm to (167.4, 81.7)
- moved Q17 67.8 mm to (181.6, 79.6)
- moved C24 67.8 mm to (181.1, 51.5)
- moved D2 67.8 mm to (167.4, 57.9)
- moved Q3 67.8 mm to (161.5, 55.5)
- moved R12 67.8 mm to (164.2, 52.5)
- moved R37 67.8 mm to (167.4, 54.2)
- moved R38 67.8 mm to (167.4, 62.0)
- moved R39 67.8 mm to (167.6, 70.1)
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Routing:
- net +5V: track 46.0 -> 5.38 mm
- net CAN_STBY: track 37.2 -> 0.00 mm
- net Net-(U4-SW): track 29.6 -> 0.00 mm
- net +3.3V: track 108.1 -> 83.5 mm
- net CAN1_TX: track 24.5 -> 0.00 mm
- net CAN1_RX: track 23.8 -> 0.00 mm
- net CAN1+: track 13.6 -> 0.00 mm
- net SWDCLK: track 12.1 -> 0.00 mm
- net CAN1-: track 11.5 -> 0.00 mm
- net UART_RX: track 11.3 -> 0.00 mm
- net SWDIO: track 10.9 -> 0.00 mm
- net UART_TX: track 10.5 -> 0.00 mm
- net VIN: track 21.2 -> 11.1 mm
- net CL4_DCH: track 7.24 -> 0.00 mm
- net Net-(Q13-B): track 6.68 -> 0.00 mm
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